File: EDAFiles/KiCAD_SCH/auxModule/auxModule/auxModule.kicad_sch (KiCad schematic)
At the start: 4 parts, among them J1 STX-3000, J2 6130XX243121_613010243121

Commit message: Periodic Update from local Machine
Connections:
- net filament+: now also J2.7, J2.8; no longer J2.5, J2.6
- net filament-: now also J2.5, J2.6; no longer J2.7, J2.8
- net at J2.10, J2.9: now also R1.2, R2.1; no longer R1.1, R2.2
- net at J1.2: now also R1.1; no longer R1.2
- net at J1.3: now also R2.2; no longer R2.1
Other:
- moved on the sheet: R1, R2
Changed lines of the file:
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@@
 		)
 	)
-	(global_label "filament-"
+	(global_label "filament+"
 		(shape input)
 		(at 130.81 97.79 270)
@@
 		)
 	)
-	(global_label "filament+"
+	(global_label "filament-"
 		(shape input)
 		(at 134.62 97.79 270)
@@
 	(symbol
 		(lib_id "Device:R_US")
-		(at 88.9 71.12 270)
+		(at 88.9 71.12 90)
 		(unit 1)
 		(exclude_from_sim no)
@@
 		)
 		(property "Footprint" "Resistor_THT:R_Axial_DIN0207_L6.3mm_D2.5mm_P10.16mm_Horizontal"
-			(at 88.646 72.136 90)
+			(at 89.154 70.104 90)
 			(effects
 				(font
@@
 	(symbol
 		(lib_id "Device:R_US")
-		(at 88.9 82.55 90)
-		(unit 1)
-		(exclude_from_sim no)
-		(in_bom yes)
-		(on_board yes)
-		(dnp no)
-		(fields_autoplaced yes)
+		(at 88.9 82.55 270)
+		(mirror x)
+		(unit 1)
+		(exclude_from_sim no)
+		(in_bom yes)
+		(on_board yes)
+		(dnp no)
 		(property "Reference" "R2"
 			(at 88.9 76.2 90)
@@
 		)
 		(property "Footprint" "Resistor_THT:R_Axial_DIN0207_L6.3mm_D2.5mm_P10.16mm_Horizontal"
-			(at 89.154 81.534 90)
-			(effects
-				(font
+			(at 88.646 81.534 90)
+			(effects
+				(font
